File: Electronics/GrooveBox.kicad_pcb (KiCad board)
At the start: 2 copper layers, 77 x 32 mm, 39 parts, among them J1 JACK_TRS_6PINS, P1 R_Potentiometer, P2 R_Potentiometer, P5 R_Potentiometer, P6 R_Potentiometer, P7 R_Potentiometer, P8 R_Potentiometer, SW1 SW_Push, SW2 SW_Push, SW3 SW_Push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

Commit message: Version sent to PCB Manufacturing Yeah
Parts:
- removed C2: 100nF, Capacitor_SMD:C_0805_2012Metric
- added G***: LOGO, GaudiLabsLogos:GaudiLabs_8, B.Cu at (137.1, 108.1)
- added G***: LOGO, GaudiLabsLogos:MirnadaEnergyCommunity, B.Cu at (127.3, 105.8)
- added R5: 10k DNP, Resistor_SMD:R_0805_2012Metric, F.Cu at (142.2, 102.8)
Connections:
- A1 pad 19: Net-(A1-Pad19) -> Net-(P1-Pad2)
- A1 pad 22: Net-(A1-Pad22) -> Net-(R4-Pad2)
- A1 pad 24: Net-(A1-Pad24) -> Net-(P6-Pad2)
- A1 pad 25: Net-(A1-Pad25) -> Net-(P7-Pad2)
- P1 pad 1: Net-(A1-Pad19) -> VCC
- P1 pad 2: unconnected-(P1-Pad2) -> Net-(P1-Pad2)
- P2 pad 1: Net-(A1-Pad20) -> VCC
- P2 pad 2: unconnected-(P2-Pad2) -> Net-(A1-Pad20)
- P5 pad 1: Net-(A1-Pad23) -> VCC
- P5 pad 2: unconnected-(P5-Pad2) -> Net-(A1-Pad23)
- P6 pad 1: Net-(A1-Pad24) -> VCC
- P6 pad 2: unconnected-(P6-Pad2) -> Net-(P6-Pad2)
- P7 pad 1: Net-(A1-Pad25) -> VCC
- P7 pad 2: unconnected-(P7-Pad2) -> Net-(P7-Pad2)
- P8 pad 1: Net-(A1-Pad26) -> VCC
- P8 pad 2: unconnected-(P8-Pad2) -> Net-(A1-Pad26)
- R3 pad 1: Net-(A1-Pad21) -> VCC
- R3 pad 2: unconnected-(R3-Pad2) -> Net-(A1-Pad21)
- R4 pad 1: Net-(A1-Pad22) -> VCC
- R4 pad 2: unconnected-(R4-Pad2) -> Net-(R4-Pad2)
Routing:
- net VCC: track 88.1 -> 178.2 mm, vias 1 -> 2
- net Net-(A1-Pad25): track 28.2 -> 0.00 mm, vias 1 -> 0
- net Net-(P7-Pad2): track 0.00 -> 27.3 mm, vias 0 -> 1
- net Net-(A1-Pad24): track 26.8 -> 0.00 mm, vias 1 -> 0
- net Net-(A1-Pad22): track 25.0 -> 0.00 mm, vias 1 -> 0
- net Net-(P6-Pad2): track 0.00 -> 24.0 mm, vias 0 -> 1
- net Net-(A1-Pad19): track 23.4 -> 0.00 mm, vias 1 -> 0
- net Net-(R4-Pad2): track 0.00 -> 12.8 mm, vias 0 -> 1
- net Net-(A1-Pad21): track 22.5 -> 9.76 mm
- net Net-(A1-Pad20): track 22.0 -> 10.0 mm
- net Net-(P1-Pad2): track 0.00 -> 8.52 mm, vias 0 -> 1
- net GND: track 35.2 -> 43.2 mm, vias 12 -> 16
- net Net-(A1-Pad23): track 25.4 -> 17.8 mm
- net unconnected-(P8-Pad2): track 3.60 -> 0.00 mm
- net unconnected-(R4-Pad2): track 3.60 -> 0.00 mm
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Other:
- board text added: "Arduino-Nano"
- board text added: "Mozzi Library"
