File: Electronics/GrooveBox.kicad_sch (KiCad schematic)
At the start: 38 parts, among them J1 JACK_TRS_6PINS, P1 R_Potentiometer, P2 R_Potentiometer, P5 R_Potentiometer, P6 R_Potentiometer, P7 R_Potentiometer, P8 R_Potentiometer, SW1 SW_Push, SW2 SW_Push, SW3 SW_Push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

Commit message: Version sent to PCB Manufacturing Yeah
Parts:
- removed C2: 100nF, Capacitor_SMD:C_0805_2012Metric, symbol Device:C
- added R5: 10k DNP, Resistor_SMD:R_0805_2012Metric, symbol Device:R
Connections:
- net VCC: now also P1.1, P2.1, P5.1, P6.1, P7.1, P8.1, R3.1, R4.1, R5.2
- net at A1.26 (A7): now also P8.2; no longer P8.1
- net at A1.19 (A0): now also P1.2; no longer P1.1
- net at A1.23 (A4): now also P5.2; no longer P5.1
- net at A1.25 (A6): now also P7.2; no longer P7.1
- net at A1.21 (A2): now also R3.2; no longer R3.1
- net at A1.22 (A3): now also R4.2; no longer R4.1
- net at A1.28 (~{RESET}), A1.3 (~{RESET}): now also R5.1
- net at A1.24 (A5): now also P6.2; no longer P6.1
- net at A1.20 (A1): now also P2.2; no longer P2.1
Other:
- note added: "Arduino Nano"
- note removed: "Analog Multiplexed Charge Amplifier"
- note removed: "USB-C Interface"
